Commit message: special_moveit_config now uses cob3-3-macro and moveit-param-remap for robot_description

File: special_moveit_config/config/description.urdf.xacro (robot description, xacro)
@@ -6,25 +6,12 @@
        name="cob3_3" >
   <!-- common stuff -->
-  <include filename="$(find cob_description)/urdf/common.xacro" />
-  <include filename="$(find cob_description)/urdf/materials.urdf.xacro" />
-  <include filename="$(find schunk_description)/urdf/materials.urdf.xacro" />
-  <!-- calibration -->
-  <include filename="$(find cob_calibration_data)/cob3-3/calibration/calibration.urdf.xacro" />
-  <!-- base -->
-  <include filename="$(find cob_description)/urdf/base/base.urdf.xacro" />
+  <include filename="$(find cob_hardware_config)/cob3-3/urdf/cob3-3-macro.urdf.xacro" />
+  <!-- base_placement -->
+<!--
   <include filename="$(find cob_description)/urdf/base_placement/base_placement.urdf.xacro"/>
-  <!-- tray -->
-  <include filename="$(find cob_description)/urdf/tray/tray.urdf.xacro" />
-  <!-- torso -->
-  <include filename="$(find cob_description)/urdf/torso_v1/torso.urdf.xacro" />
-  <!-- head -->
-  <include filename="$(find cob_description)/urdf/head_v3/head.urdf.xacro" />
+-->
+  <!-- lookat -->
   <include filename="$(find cob_description)/urdf/lookat/lookat.urdf.xacro" />
-  <!-- arm -->
-  <include filename="$(find cob_description)/urdf/lbr/lbr.urdf.xacro" />
-  <!-- sdh -->
-  <include filename="$(find schunk_description)/urdf/sdh/sdh.urdf.xacro" />
-  <!-- generic simulator_gazebo plugins for starting mechanism control, ros time, ros battery -->
-  <include filename="$(find cob_description)/gazebo/gazebo.urdf.xacro" />
+<!--
   <xacro:cob_base_placement name="base_placement"/>
   <joint name="base_placement_helper_joint" type="fixed">
@@ -32,25 +19,10 @@
     <child link="base_footprint"/>
   </joint>
+-->
   <!-- composition of the robot -->
-  <xacro:cob_base name="base"/>
-  <!--<xacro:cob_component type="cob_torso_v1" name="tray" parent="base_link"/>-->
-  <xacro:cob_tray name="tray" parent="base_link">
-    <origin xyz="${tray_x} ${tray_y} ${tray_z}" rpy="${tray_roll} ${tray_pitch} ${tray_yaw}" />
-  </xacro:cob_tray>
-  <xacro:cob_torso_v1 name="torso" parent="base_link">
-    <origin xyz="${torso_x} ${torso_y} ${torso_z}" rpy="${torso_roll} ${torso_pitch} ${torso_yaw}" />
-  </xacro:cob_torso_v1>
-  <xacro:cob_lbr name="arm" parent="base_link">
-    <origin xyz="${arm_x} ${arm_y} ${arm_z}" rpy="${arm_roll} ${arm_pitch} ${arm_yaw}" />
-  </xacro:cob_lbr>
-  <xacro:cob_head_v3 name="head" parent="torso_upper_neck_tilt_link">
-    <origin xyz="${head_x} ${head_y} ${head_z}" rpy="${head_roll} ${head_pitch} ${head_yaw}" />
-  </xacro:cob_head_v3>
+  <xacro:cob3-3/>
   <xacro:cob_lookat name="lookat" parent="torso_upper_neck_tilt_link">
     <origin xyz="${head_x} ${head_y} ${head_z}" rpy="${head_roll} ${head_pitch} ${head_yaw}" />
     <axis xyz="-1 0 0"/>
   </xacro:cob_lookat>
-  <xacro:schunk_sdh name="sdh" parent="arm_7_link">
-    <origin xyz="${sdh_x} ${sdh_y} ${sdh_z}" rpy="${sdh_roll} ${sdh_pitch} ${sdh_yaw}" />
-  </xacro:schunk_sdh>
 </robot>
